Commit message: switched to flex physics backend

File: assets/urdf/dvrk_description/psm/psm_for_issacgym.urdf (robot description, URDF)
Before this commit: robot psm, 12 links, 11 joints
Joints:
- joint psm_rev_joint: limit lower=0 upper=0 effort=1000 velocity=10 -> lower=0 upper=0 effort=100 velocity=10

Commit message: update

File: assets/urdf/dvrk_description/psm/psm_for_issacgym.urdf (robot description, URDF)
Before this commit: robot psm, 12 links, 11 joints
Joints:
- joint psm_main_insertion_joint: limit lower=0.042 upper=0.24 effort=1000.0 velocity=0.1 -> lower=0.042 upper=0.24 effort=100.0 velocity=0.1
- joint psm_pitch_back_joint: limit lower=-0.93556 upper=0.94249 effort=1000.0 velocity=10.0 -> lower=-0.93556 upper=0.94249 effort=100.0 velocity=10.0
- joint psm_pitch_bottom_joint: limit lower=-0.94249 upper=0.93556 effort=1000.0 velocity=10.0 -> lower=-0.94249 upper=0.93556 effort=100.0 velocity=10.0
- joint psm_pitch_end_joint: limit lower=-0.93556 upper=0.94249 effort=1000.0 velocity=10.0 -> lower=-0.93556 upper=0.94249 effort=100.0 velocity=10.0
- joint psm_tool_pitch_joint: limit lower=-1.5708 upper=1.5708 effort=1000.0 velocity=10.0 -> lower=-1.5708 upper=1.5708 effort=100.0 velocity=10.0
- joint psm_tool_roll_joint: limit lower=-3.14 upper=3.14 effort=1000.0 velocity=10.0 -> lower=-3.14 upper=3.14 effort=100.0 velocity=10.0
- joint psm_tool_yaw_joint: limit lower=-1.5708 upper=1.5708 effort=1000.0 velocity=10.0 -> lower=-1.5708 upper=1.5708 effort=100.0 velocity=10.0
- joint psm_yaw_joint: limit lower=-1.605 upper=1.5994 effort=1000.0 velocity=10.0 -> lower=-1.605 upper=1.5994 effort=100.0 velocity=10.0

Commit message: liver assets

File: assets/urdf/dvrk_description/psm/psm_for_issacgym.urdf (robot description, URDF)
Before this commit: robot psm, 12 links, 11 joints
Joints:
- joint psm_tool_gripper1_joint: limit lower=-10.0 upper=20.0 effort=10 velocity=1 -> lower=0 upper=1.5707 effort=10 velocity=1
- joint psm_tool_gripper2_joint: limit lower=-10.0 upper=20.0 effort=10 velocity=1 -> lower=0 upper=1.5707 effort=10 velocity=1
